Commit message: Implemented action server for GraspPlanner
It seems that Moveit was not able to add collision objects (the ground plane)
to the planning scene when the respective nodes were not launched in the
namespace were Moveit was launched. This needs further investigation.

File: chair_manipulation_gazebo/urdf/kinect/kinect.urdf.xacro (robot description, xacro)
@@ -43,10 +43,10 @@
 				</geometry>
 			</visual>
-			<collision>
+			<!-- <collision>
 				<origin xyz="0.0 0.0 0.0" rpy="0 0 0"/>
 				<geometry>
 					<box size="0.07271 0.27794 0.073"/>
 				</geometry>
-			</collision>
+			</collision> -->
 			<inertial>
 				<mass value="0.001" />

Commit message: Remove common sensors dependency

File: chair_manipulation_gazebo/urdf/kinect/kinect.urdf.xacro (robot description, xacro)
@@ -40,5 +40,5 @@
 			 <origin xyz="0 0 0" rpy="0 0 ${pi/2}"/>
 				<geometry>
-				<mesh filename="package://common_sensors/meshes/sensors/kinect.dae"/>
+				<mesh filename="package://chair_manipulation_gazebo/meshes/sensors/kinect.dae"/>
 				</geometry>
 			</visual>
